File: top-plate/top-plate.kicad_pcb (KiCad board)
At the start: 2 copper layers, 309.8 x 119.3 mm, 4 parts

Commit message: Top plate: KS-33 cut-outs, Gateron 6.25U stabiliser cut-out, 1.2 mm
Switch cut-outs are 14.00 mm squares (Gateron KS-33 drawing) at the
new switch positions, including the HHKB Pro 2 bottom row. The space
bar cut-out is merged with Gateron's recommended KS-57B623T stabiliser
cut-out at 100 mm stem spacing, notch facing the back to match the PCB
slots. Board thickness set to 1.2 mm (KS-33 and stabiliser drawings).
Outline and M2 holes unchanged. DRC: 0 violations.

Co-Authored-By: Claude Opus 5.5 <noreply@anthropic.com>
Claude-Session: https://claude.ai/code/session_011sJxCFL16sEAYrBmNTBwJC
Parts:
- removed REF** (x4): STAB_choc_2u_plate, local:STAB_choc_2u_plate
Other:
- outline, holes or cut-outs redrawn
