File: boethia60/boethia60.kicad_pcb (KiCad board)
At the start: 2 copper layers, 287.3 x 98.4 mm, 161 parts, among them J1 Conn_01x06, SW1 SW_Push, U1 NCP1117-3.3_SOT223, U2 PRTR5V0U2X, U3 RP2040, U4 W25Q128JVS, Y1 Crystal_GND24_Small

Commit message: PCB (work in progress): KS-33 footprints, HHKB bottom row, matrix rerouted
Not finished: 4 matrix connections still open (col0, col10, col14, row3);
DRC otherwise reports only the two pre-existing USB1 pad clearances plus
two to review. Factory files are not regenerated yet.

- 60 KS-33 hot-swap footprints, sockets on the underside; 55 rotated 180
  degrees so the diode pad faces the diode (K_14, K_15, K_29, K_42, K_55
  stay at 0 next to the USB connector)
- K_58/D_58/K_60/D_60 removed; bottom row moved per HANDOVER.md section 5
- Gateron 6.25U stabiliser slots (ST1), wire-hook side to the back
- original row/column routing kept where it does not clash; the rest
  routed by a grid router; default net class 0.2/0.15 mm, via 0.6/0.3
- 16 USB/power segments displaced by the new sockets rerouted; +3V3 now
  takes the lane of a redundant GND edge track (GND is poured)

Co-Authored-By: Claude Opus 5.5 <noreply@anthropic.com>
Claude-Session: https://claude.ai/code/session_011sJxCFL16sEAYrBmNTBwJC
Parts:
- removed D_58, D_60: D, Diode_SMD:D_SOD-323
- removed K_58, K_60: space, local:SW_Hotswap_Kailh_Choc_V1V2_annotated
- removed REF** (x4): STAB_choc_2u, PCM_marbastlib-xp-choc:STAB_choc_2u
- added ST1: KS-57B623T, local:STAB_Gateron_LP_6.25U_PCB, F.Cu at (154.8, 85.7)
- K_1, K_10, K_11, K_12, K_13, K_14, K_15, K_17, K_18, K_19, K_2, K_20, K_21, K_22, K_23, K_24, K_25, K_26, K_27, K_28, K_3, K_31, K_32, K_33, K_34, K_35, K_36, K_37, K_38, K_39, K_4, K_40, K_41, K_42, K_43, K_44, K_45, K_46, K_47, K_48, K_49, K_5, K_50, K_51, K_52, K_53, K_55, K_56, K_59, K_6, K_62, K_7, K_8, K_9: footprint local:SW_Hotswap_Kailh_Choc_V1V2_annotated -> marbastlib-xp-gateron_lp:SW_KS33_HS_KS-2P02B01-02_HS_1u; moved to F.Cu
- K_16, K_29, K_57, K_61: footprint local:SW_Hotswap_Kailh_Choc_V1V2_annotated -> marbastlib-xp-gateron_lp:SW_KS33_HS_KS-2P02B01-02_1.5u; moved to F.Cu
- K_30, K_54: footprint local:SW_Hotswap_Kailh_Choc_V1V2_annotated -> marbastlib-xp-gateron_lp:SW_KS33_HS_KS-2P02B01-02_1.75u; moved to F.Cu
- moved K_56 4.76 mm to (252.4, 85.7), turned to 180 degrees
- moved D_56 4.76 mm to (261.1, 83.3)
- moved K_57 4.76 mm to (228.6, 85.7), turned to 180 degrees
- moved D_57 4.76 mm to (237.3, 83.3)
- moved D_1 2.51 mm to (285.0, 7.14), turned to -90 degrees
- moved K_59 2.38 mm to (154.8, 85.7), turned to 180 degrees
- moved D_59 2.38 mm to (163.5, 83.3)
- moved D_15 2.27 mm to (18.3, 18.4)
- turned K_1 to 180 degrees
- turned K_10 to 180 degrees
- turned K_11 to 180 degrees
- turned K_12 to 180 degrees
- turned K_13 to 180 degrees
- turned K_16 to 180 degrees
- turned K_17 to 180 degrees
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Routing:
- net col0: track 325.4 -> 61.5 mm, vias 4 -> 3
- net row0: track 592.8 -> 349.2 mm, vias 2 -> 20
- net col10: track 164.7 -> 92.4 mm, vias 6 -> 5
- net GND: track 260.4 -> 199.7 mm, vias 27 -> 24
- net row1: track 565.2 -> 621.2 mm, vias 2 -> 4
- net col14: track 83.2 -> 30.1 mm, vias 4 -> 1
- net row2: track 287.8 -> 336.9 mm, vias 0 -> 4
- net col5: track 268.7 -> 253.7 mm, vias 6 -> 7
- net col13: track 95.4 -> 80.7 mm, vias 4 -> 2
- net row4: track 271.9 -> 284.8 mm, vias 0 -> 6
- net col1: track 309.9 -> 322.1 mm, vias 2 -> 4
- net DN: track 96.9 -> 87.2 mm, vias 0 -> 4
- net col3: track 291.6 -> 300.7 mm, vias 5 -> 4
- net Net-(D_55-A): track 2.05 -> 11.1 mm, vias 0 -> 1
- net Net-(D_29-A): track 2.05 -> 11.0 mm
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