File: boethia60/boethia60.kicad_pcb (KiCad board)
At the start: 2 copper layers, 287.3 x 98.4 mm, 154 parts, among them J1 Conn_01x06, SW1 SW_Push, U1 NCP1117-3.3_SOT223, U2 PRTR5V0U2X, U3 RP2040, U4 W25Q128JVS, Y1 Crystal_GND24_Small

Commit message: PCB: finish matrix routing
Close the last four links by hand (row 3, col 0, col 10, col 14). Col 0
leaves its old y 76.5 mm lane, which crosses both stabiliser slots, and
runs under the row 3 switches instead; col 9 drops one lane beside the
RP2040 to make room for a col 0 via. Remove dead-end vias and stubs left
from the original routing. DRC: 0 unconnected pads; only the two
pre-existing USB1 pad clearances remain.

Co-Authored-By: Claude Opus 5.5 <noreply@anthropic.com>
Claude-Session: https://claude.ai/code/session_011sJxCFL16sEAYrBmNTBwJC
Routing:
- net col0: track 61.5 -> 343.2 mm, vias 3 -> 12
- net col10: track 92.4 -> 160.5 mm, vias 5 -> 4
- net col14: track 30.1 -> 68.8 mm, vias 1 -> 4
- net row3: track 293.2 -> 324.9 mm, vias 5 -> 9
- net col5: track 253.7 -> 234.3 mm, vias 7 -> 3
- net col11: track 131.4 -> 130.8 mm, vias 8 -> 6
- net col3: track 300.7 -> 300.3 mm, vias 4 -> 3
- net col9: track 163.8 -> 164.2 mm, vias 9 -> 6
- net col12: track 135.8 -> 135.6 mm, vias 4 -> 2
- net col8: track 207.5 -> 207.3 mm, vias 8 -> 5
- net col7: vias 9 -> 6
- net col6: vias 6 -> 3
- net col2: vias 4 -> 3

Commit message: Fuse, part labels, Polymetis name
- F1: the original BOM fitted a ferrite bead (C1015) where the schematic
  has a 500 mA fuse; now SMD0805P050TF/12 (C90129, 500 mA hold, 1 A
  trip, 12 V) on the same 0805 footprint, which carries its terminals.
- Labels match the fitted parts: U1 XC6206P332MR, U4 W25Q16JVSSIQ,
  FB1 120@100MHz (BLM18PG121SN1D), with datasheet links.
- Board text: Polymetis, based on boethia60 by arviceblot, moved clear
  of D_56 and rev1, in KiCad's stroke font.
- USB product name, Vial and KLE layout names: Polymetis.

Co-Authored-By: Claude Opus 5.5 <noreply@anthropic.com>
Claude-Session: https://claude.ai/code/session_011sJxCFL16sEAYrBmNTBwJC
Parts:
- FB1: value 60@100MHz -> 120@100MHz
- U1: value NCP1117-3.3_SOT223 -> XC6206P332MR
- U4: value W25Q128JVS -> W25Q16JVSSIQ
Other:
- board text added: "Polymetis"
- board text added: "based on boethia60 by arviceblot"
- board text removed: "boethia60"
- board text removed: "by arviceblot"
