File: boethia60/boethia60.kicad_sch (KiCad schematic)
At the start: 157 parts, among them J1 Conn_01x06, SW1 SW_Push, U1 NCP1117-3.3_SOT223, U2 PRTR5V0U2X, U3 RP2040, U4 W25Q128JVS, Y1 Crystal_GND24_Small

Commit message: Schematic: KS-33 hot-swap footprints, remove split-spacebar switches
All 60 switch symbols now use the marbastlib KS-33 / KS-2P02B01-02
hot-swap footprints (1.5u and 1.75u variants for Tab, Backspace, Cmd,
Ctrl and right Shift; 1u elsewhere, including the 2.25u and 6.25u keys).
K_58, D_58, K_60 and D_60 and their wires are deleted; the space bar
keeps K_59 at matrix position (4,6). ERC reports nothing new; the
remaining items are pre-existing in the RP2040 section.

Also adds the board-only footprint for the Gateron 6.25U stabiliser
PCB slots (6.5 x 16 mm at 100 mm spacing, after Keebio's slot).

Co-Authored-By: Claude Opus 5.5 <noreply@anthropic.com>
Claude-Session: https://claude.ai/code/session_011sJxCFL16sEAYrBmNTBwJC
Parts:
- removed D_58, D_60: D, Diode_SMD:D_SOD-323, symbol Device:D_Small
- removed K_58, K_60: space, local:SW_Hotswap_Kailh_Choc_V1V2_annotated, symbol MX_Alps_Hybrid:MX-NoLED
- K_1, K_10, K_11, K_12, K_13, K_14, K_15, K_17, K_18, K_19, K_2, K_20, K_21, K_22, K_23, K_24, K_25, K_26, K_27, K_28, K_3, K_31, K_32, K_33, K_34, K_35, K_36, K_37, K_38, K_39, K_4, K_40, K_41, K_42, K_43, K_44, K_45, K_46, K_47, K_48, K_49, K_5, K_50, K_51, K_52, K_53, K_55, K_56, K_59, K_6, K_62, K_7, K_8, K_9: footprint local:SW_Hotswap_Kailh_Choc_V1V2_annotated -> marbastlib-xp-gateron_lp:SW_KS33_HS_KS-2P02B01-02_HS_1u
- K_16, K_29, K_57, K_61: footprint local:SW_Hotswap_Kailh_Choc_V1V2_annotated -> marbastlib-xp-gateron_lp:SW_KS33_HS_KS-2P02B01-02_1.5u
- K_30, K_54: footprint local:SW_Hotswap_Kailh_Choc_V1V2_annotated -> marbastlib-xp-gateron_lp:SW_KS33_HS_KS-2P02B01-02_1.75u

Commit message: BOM: flash U4 to C131025 (same W25Q16JVSSIQ, in stock)
C82317 has 8 left at JLCPCB; C131025 is the same Winbond part in the
same SOIC-8 208-mil package with 1,317 in stock.

Co-Authored-By: Claude Opus 5.5 <noreply@anthropic.com>
Claude-Session: https://claude.ai/code/session_011sJxCFL16sEAYrBmNTBwJC
Parts:
- U4: JLCPCB Part C82317 -> C131025
Changed lines of the file:
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@@
 			)
 		)
-		(property "JLCPCB Part" "C82317"
+		(property "JLCPCB Part" "C131025"
 			(at 262.89 274.32 0)
 			(effects

Commit message: Fuse, part labels, Polymetis name
- F1: the original BOM fitted a ferrite bead (C1015) where the schematic
  has a 500 mA fuse; now SMD0805P050TF/12 (C90129, 500 mA hold, 1 A
  trip, 12 V) on the same 0805 footprint, which carries its terminals.
- Labels match the fitted parts: U1 XC6206P332MR, U4 W25Q16JVSSIQ,
  FB1 120@100MHz (BLM18PG121SN1D), with datasheet links.
- Board text: Polymetis, based on boethia60 by arviceblot, moved clear
  of D_56 and rev1, in KiCad's stroke font.
- USB product name, Vial and KLE layout names: Polymetis.

Co-Authored-By: Claude Opus 5.5 <noreply@anthropic.com>
Claude-Session: https://claude.ai/code/session_011sJxCFL16sEAYrBmNTBwJC
Parts:
- F1: JLCPCB Part C1015 -> C90129
- FB1: value 60@100MHz -> 120@100MHz
- U1: value NCP1117-3.3_SOT223 -> XC6206P332MR
- U4: value W25Q128JVS -> W25Q16JVSSIQ
Changed lines of the file:
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@@
 			)
 		)
-		(property "Value" "60@100MHz"
+		(property "Value" "120@100MHz"
 			(at 215.8619 187.96 90)
 			(effects
@@
 			)
 		)
-		(property "Datasheet" "~"
+		(property "Datasheet" "https://www.lcsc.com/datasheet/lcsc_datasheet_2304140030_Murata-Electronics-BLM18PG121SN1D_C14709.pdf"
 			(at 215.9 191.77 0)
 			(effects
@@
 			)
 		)
-		(property "Value" "W25Q128JVS"
+		(property "Value" "W25Q16JVSSIQ"
 			(at 271.78 275.5899 0)
 			(effects
@@
 			)
 		)
-		(property "Datasheet" "https://www.winbond.com/resource-files/w25q128jv_dtr%20revc%2003272018%20plus.pdf"
+		(property "Datasheet" "~"
 			(at 262.89 248.92 0)
 			(effects
@@
 			)
 		)
-		(property "Value" "NCP1117-3.3_SOT223"
+		(property "Value" "XC6206P332MR"
 			(at 195.58 161.29 0)
 			(effects
@@
 			)
 		)
-		(property "Datasheet" "http://www.onsemi.com/pub_link/Collateral/NCP1117-D.PDF"
+		(property "Datasheet" "https://www.lcsc.com/datasheet/lcsc_datasheet_2304140030_Torex-Semicon-XC6206P332MR-G_C5446.pdf"
 			(at 198.12 171.45 0)
 			(effects
@@
 			)
 		)
-		(property "Datasheet" "~"
+		(property "Datasheet" "https://www.lcsc.com/datasheet/lcsc_datasheet_2403081022_RUILON-Shenzhen-Ruilongyuan-Elec-SMD0805P050TF-12_C90129.pdf"
 			(at 147.32 165.1 0)
 			(effects
@@
 			)
 		)
-		(property "JLCPCB Part" "C1015"
+		(property "JLCPCB Part" "C90129"
 			(at 147.32 165.1 0)
 			(effects
