File: pcb/polymetis.kicad_pcb (KiCad board)
At the start: 2 copper layers, 287.3 x 98.4 mm, 154 parts, among them J1 Conn_01x06, SW1 SW_Push, U1 XC6206P332MR, U2 PRTR5V0U2X, U3 RP2040, U4 W25Q16JVSSIQ, Y1 Crystal_GND24_Small

Commit message: Drop references to the original design; dark grey modifier keycaps
- Main PCB project moves to pcb/polymetis.*; firmware crate, KLE layout,
  factory files, check reports and UF2 are named polymetis.
- Board text: the credit line is removed. Bottom plate: the old logo is
  replaced by Polymetis text on the outside face.
- Unused legacy files removed: KiCad 5 project, kbplacer log, FreeCAD
  frame, plate-generator outlines, the original handover brief. The
  frame script reads case/frame-source.stl.
- README, HANDOVER and CLAUDE.md no longer describe Polymetis as a fork.
  LICENSE is unchanged: the MIT terms require its copyright and
  permission notice to stay with the design.
- Keycaps: a sixth colour, dark grey (the body colour), for the 11
  modifiers; the layout page, concept model, layout image and renders
  are updated.

Co-Authored-By: Claude Opus 5.5 <noreply@anthropic.com>
Claude-Session: https://claude.ai/code/session_011sJxCFL16sEAYrBmNTBwJC
Other:
- board text removed: "based on boethia60 by arviceblot"
Changed lines of the file:
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@@
 		(layer "Edge.Cuts")
-	)
-	(gr_text "based on boethia60 by arviceblot"
-		(at 262.5 91.4 0)
-		(layer "F.SilkS")
-		(effects
-			(font
-				(size 0.8 0.8)
-				(thickness 0.12)
-			)
-			(justify left bottom)
-		)
 	)
 	(gr_text "rev1"
